File: FrontEnd/DualMixer/Converter_Head/Converter_Head.sch (KiCad schematic (older format))
At the start: 0 parts

Commit message: Added power, needs to add communication connector
Parts:
- added C101, C102, C118, C119: 10u, SM1206, symbol passives:CAP_1206
- added C103, C104, C110, C111: 10uF, SM0805, symbol passives:CAP_0805
- added C105, C117: 470p, SM0603, symbol passives:CAP_0603
- added C106, C115: 47n, SM0603, symbol passives:CAP_0603
- added C107: 2.8n, SM0603, symbol passives:CAP_0603
- added C108, C109: 1nF, SM0603, symbol passives:CAP_0603
- added C112: 4.7u, SM0603, symbol passives:CAP_0603
- added C113, C116: 10uF, SM1206, symbol passives:CAP_1206
- added C114: 1.68n, SM0603, symbol passives:CAP_0603
- added C120, C121, C122, C123, C127, C128, C129, C130, C131: 0.1uF, SM0402, symbol passives:CAP_0402
- added C124, C125: 100nF, SM0402, symbol passives:CAP_0402
- added C126: 10nF, SM0402, symbol passives:CAP_0402
- added J101: Conn_01x03, Connectors_POWER:2.1mm_DC_Jack_NEB21R, symbol Connector_Generic:Conn_01x03
- added J102: SMA_PCB, symbol RF_Connectors:SMA_PCB
- added L101, L102: 5.6uH, Wurth:WE-HCI_SMD_5.6x5.3x4, symbol passives:IND_SMALL
- added L103: IND_0603, SM0603, symbol passives:IND_0603
- added L104: IND_0402, SM0402, symbol passives:IND_0402
- added OC101: ECOC-2522-40.000-3GS, symbol ECOC-2522:ECOC-2522-40.000-3GS
- added Q101: BSS138, SOT:SOT-23, symbol NMOS:BSS138
- added R101, R110: 0, General_SMD:SM1206, symbol passives:RES_1206
- added R102, R108: 20.5k, SM0603, symbol passives:RES_0603
- added R103: 3.48k, SM0603, symbol passives:RES_0603
- added R104, R107: 10, SM0603, symbol passives:RES_0603
- added R105: 34.8k, SM0603, symbol passives:RES_0603
- added R106: 57.6k, SM0603, symbol passives:RES_0603
- added R109: 6.49k, SM0603, symbol passives:RES_0603
- added R111, R112: 10k, SM0603, symbol passives:RES_0603
- added R113: RVAR, symbol passives:RVAR
- added R114, R115, R120: NC, SM0402, symbol passives:RES_0402
- added R116: 50, SM0402, symbol passives:RES_0402
- added R117, R118, R119: 0, SM0402, symbol passives:RES_0402
- added U101, U102: ADM7170ACPZ-3.3, QFN:DFN8_3x3mm, symbol adm7170:ADM7170
- added U103: TPS54292, SSOP:PowerPad_TSSOP_16, symbol tps5429x:TPS5429x
- added U104: LTC6957IMS-3, symbol LTC6957:LTC6957IMS-3
Connections:
- net ADF4355 PLL/CLKREF_N: now also C131.1
- net ADF4355 PLL/CLKREF_P: now also U104.10 (OUT1)
- new net: R114.2, R117.1, U104.1 (FILTA)
- new net: C128.1, C129.1, L104.2, R117.2, R118.2, U104.11 (Vdd), U104.2 (V+)
- new net: C125.1, U104.3 (IN+)
- new net: C126.1, U104.4 (IN-)
- new net: R115.2, R118.1, U104.6 (FILTB)
- new net: R119.2, U104.9 (OUT2)
- new net: C130.2, J102.1 (sig)
- new net: C130.1, R119.1, R120.1
- new net: C124.1, C125.2, R116.1
- new net: C123.1, OC101.1 (Vcont), R113.2
- new net: C122.1, OC101.2 (Vref), R113.1
- new net: C121.1, L103.2, OC101.3 (Vd)
- new net: C124.2, OC101.4 (Out)
- new net: R108.2, R109.1, U103.10 (FB2)
- new net: C112.1, U103.12 (BP)
- new net: C115.2, U103.15 (BOOT2)
- new net: C106.2, U103.2 (BOOT1)
- new net: Q101.3 (D), R111.2, U103.5 (~EN1), U103.6 (~EN2)
- new net: R102.2, R103.1, U103.7 (FB1)
- new net: R105.1, U103.8 (COMP1)
- new net: R106.1, U103.9 (COMP2)
- new net: C105.2, R104.1
- new net: C107.1, R105.2
- new net: C117.2, R107.1
- new net: C114.1, R106.2
- new net: C108.1, U101.4 (SS)
- new net: C109.1, U102.4 (SS)
- new net +12V: C113.1, C116.1, J101.1 (Pin_1), R111.1, U103.1 (PVDD1), U103.16 (PVDD2)
- new net +3.3VM1: C110.1, U101.1 (Vout), U101.2 (Vout), U101.3 (Sense)
- new net +3.3VM2: C111.1, U102.1 (Vout), U102.2 (Vout), U102.3 (Sense)
- new net +3V3: C120.1, C127.1, L103.1, L104.1, R110.1
- new net +5.5V: C103.1, C104.1, R101.1, U101.5 (EN), U101.7 (Vin), U101.8 (Vin), U102.5 (EN), U102.7 (Vin), U102.8 (Vin)
- new net 2.5V_R: C101.1, C102.1, L101.1, R101.2, R102.1
- new net 2.5V_SW: C105.1, C106.1, L101.2, U103.3 (SW1)
- new net 3.3V_R: C118.1, C119.1, L102.1, R108.1, R110.2
- new net 3.3V_SW: C115.1, C117.1, L102.2, U103.14 (SW2)
- new net FRONTEND_EN: Q101.1 (G), R112.1
- new net GND: C101.2, C102.2, C103.2, C104.2, C107.2, C108.2, C109.2, C110.2, C111.2, C112.2, C113.2, C114.2, C116.2, C118.2, C119.2, C120.2, C121.2, C122.2, C123.2, C126.2, C127.2, C128.2, C129.2, C131.2, J101.2 (Pin_2), J101.3 (Pin_3), J102.2, OC101.5 (GND), Q101.2 (S), R103.2, R104.2, R107.2, R109.2, R112.2, R113.3, R114.1, R115.1, R116.2, R120.2, U101.6 (GND), U101.9 (PAD), U102.6 (GND), U102.9 (PAD), U103.11 (GND), U103.13 (PGND2), U103.17 (EP), U103.4 (PGND1), U104.12 (SD1), U104.5 (GND), U104.7 (SD2), U104.8 (GNDOUT)
Other:
- note added: "12V Input"
- note added: "3.3V @ 2.5A"
- note added: "5.5V @ 2A"
- note added: "OCXO + Clock buffer"
- note added: "RF LDOs"
- note removed: "LTC6957-3"
- note removed: "OH300-50503CF-040.0M"
- note removed: "PLUTO"

Commit message: sent in production
Parts:
- removed C120, C121, C122, C123: 0.1uF, SM0402, symbol passives:CAP_0402
- removed C124: 100nF, SM0402, symbol passives:CAP_0402
- removed L103: IND_0603, SM0603, symbol passives:IND_0603
- removed OC101: ECOC-2522-40.000-3GS, symbol ECOC-2522:ECOC-2522-40.000-3GS
- removed R113: RVAR, symbol passives:RVAR
- added C132, C133, C134, C137, C138: 0.1uF, SM0402, symbol passives:CAP_0402
- added C135, C136: 10pF, SM0402, symbol passives:CAP_0402
- added D101, D102, D103, D104: LED, General_SMD:LED-0603, symbol passives:LED
- added J103: Conn_02x06_Odd_Even, Connectors_254mm:pin_array_6x2, symbol Connector_Generic:Conn_02x06_Odd_Even
- added J104: Conn_02x03_Odd_Even, Connector_PinHeader_2.54mm:PinHeader_2x03_P2.54mm_Vertical, symbol Connector_Generic:Conn_02x03_Odd_Even
- added J105: Conn_01x06, Connector_PinHeader_2.54mm:PinHeader_1x06_P2.54mm_Vertical, symbol Connector_Generic:Conn_01x06
- added J106: External, Connectors_254mm:pin_array_6x2, symbol Connector_Generic:Conn_02x06_Odd_Even
- added J107: SMA_PCB, Connectors_RF:SMA_RA_PCB_Amphenol, symbol RF_Connectors:SMA_PCB
- added R121, R122, R123, R126, R127: 10k, SM0603, symbol passives:RES_0603
- added R124, R128, R133, R134: 100, SM0603, symbol passives:RES_0603
- added R125: 2000k, SM0603, symbol passives:RES_0603
- added R129, R130, R131, R132: 0, SM0603, symbol passives:RES_0603
- added U105: PCA9306DCT_SSOP, SSOP:SSOP8, symbol PCA9306:PCA9306DCT_SSOP
- added U106: ATmega328PB-AU, Package_QFP:TQFP-32_7x7mm_P0.8mm, symbol MCU_Microchip_ATmega:ATmega328PB-AU
- added U107: SN74LV4T125, Package_SO:TSSOP-14_4.4x5mm_P0.65mm, symbol sn74lv4t125:SN74LV4T125
- added X101: 8MHz, Xtal_SMD:xtal_3.2x2.5, symbol xtals:SMD_XTAL_small
- C125: value 100nF -> 0.1uF
- J101: footprint Connectors_POWER:2.1mm_DC_Jack_NEB21R -> Connectors_508mm:MOL_CONN_2_VH
- J102: footprint (none) -> Connectors_RF:SMA_RA_PCB_Amphenol
- U104: footprint (none) -> Package_SO:MSOP-12_3x4mm_P0.65mm
Connections:
- net +3V3: now also C133.1, C134.1, C138.1, J104.2 (Pin_2), J106.2 (Pin_2), R121.2, R125.2, R126.2, R127.2, U106.18 (AVCC), U106.20 (AREF), U106.4 (VCC), U107.14 (Vcc)
- net +5.5V: now also J106.1 (Pin_1)
- net GND: now also C132.2, C133.2, C134.2, C135.2, C136.2, C138.2, J103.11 (Pin_11), J104.6 (Pin_6), J106.11 (Pin_11), J106.12 (Pin_12), J107.2, R124.1, R128.1, R133.1, R134.1, U105.1 (GND), U106.21 (GND), U106.5 (GND), U107.1 (~OE1), U107.10 (~OE3), U107.13 (~OE4), U107.4 (~OE2), U107.7 (GND), X101.2, X101.4
- net at C125.2, R116.1: now also C137.1
- net FRONTEND_EN renamed MIO49_FrontEnd_EN
- net MIO49_FrontEnd_EN: now also J103.5 (Pin_5)
- new net: J105.5 (Pin_5), U106.10 (PD6)
- new net: J105.6 (Pin_6), U106.11 (PD7)
- new net: D103.A, U106.19 (PE2)
- new net: D104.A, U106.22 (PE3)
- new net: J105.1 (Pin_1), U106.23 (PC0)
- new net: J105.2 (Pin_2), U106.24 (PC1)
- new net: J105.3 (Pin_3), U106.25 (PC2)
- new net: J105.4 (Pin_4), U106.26 (PC3)
- new net: D101.A, U106.3 (PE0)
- new net: D102.A, U106.6 (PE1)
- new net: C136.1, U106.7 (XTAL1/PB6), X101.3
- new net: C135.1, U106.8 (XTAL2/PB7), X101.1
- new net: R127.1, R130.2, R132.2, U105.5 (SDA2)
- new net: R126.1, R129.1, R131.1, U105.6 (SCL2)
- new net: R125.1, U105.7 (VREF2), U105.8 (EN)
- new net: C137.2, J107.1 (sig)
- new net: J106.3 (Pin_3), U107.3 (1Y)
- new net: J106.5 (Pin_5), U107.6 (2Y)
- new net: J106.7 (Pin_7), U107.8 (3Y)
- new net: J106.9 (Pin_9), U107.11 (4Y)
- new net: D104.K, R134.2
- new net: D103.K, R133.2
- new net: D102.K, R128.2
- new net: D101.K, R124.2
- new net +1.8V: C132.1, J103.12 (Pin_12), R122.2, R123.2, U105.2 (VREF1)
- new net External_CS: J106.4 (Pin_4), U106.12 (PB0)
- new net L10P: J103.1 (Pin_1), U107.2 (1A)
- new net L12N: J103.3 (Pin_3), U107.5 (2A)
- new net L24N: J103.2 (Pin_2)
- new net M1_EN: U106.32 (PD2)
- new net M1_X2: U106.1 (PD3)
- new net M2_EN: U106.2 (PD4)
- new net M2_X2: U106.9 (PD5)
- new net MIO0: J103.10 (Pin_10)
- new net MIO09: J103.7 (Pin_7)
- new net MIO10_SCL: J103.9 (Pin_9), R122.1, U105.3 (SCL1)
- new net MIO11_SDA: J103.8 (Pin_8), R123.1, U105.4 (SDA1)
- new net MIO48: J103.4 (Pin_4), U107.9 (3A)
- new net MIO53: J103.6 (Pin_6), U107.12 (4A)
- new net MISO: J104.1 (Pin_1), J106.8 (Pin_8), U106.16 (PB4)
- new net MOSI: J104.4 (Pin_4), J106.6 (Pin_6), U106.15 (PB3)
- new net PLL_LOCK: U106.13 (PB1)
- new net RXD: R131.2, U106.30 (PD0)
- new net SCK: J104.3 (Pin_3), J106.10 (Pin_10), U106.17 (PB5)
- new net SCL: R129.2, U106.28 (PC5)
- new net SDA: R130.1, U106.27 (PC4)
- new net TXD: R132.1, U106.31 (PD1)
- new net ~PLL_CS: U106.14 (PB2)
- new net ~RESET: J104.5 (Pin_5), R121.1, U106.29 (~RESET~/PC6)
Other:
- note added: "23.3mm between SMA center"
