File: FrontEnd/DualMixer/Converter_Head/mixer_1.sch (KiCad schematic (older format))
At the start: 16 parts

Commit message: Added power, needs to add communication connector
Parts:
- gave numbers to parts that had none: 16
Connections:
- net +3.3VA renamed +3.3VM1
Changed lines of the file:
@@
 $EndDescr
 $Comp
-L power:GND #PWR?
+L power:GND #PWR0159
 U 1 1 5B3C2809
 P 7075 3925
-F 0 "#PWR?" H 7075 3675 50  0001 C CNN
+F 0 "#PWR0159" H 7075 3675 50  0001 C CNN
 F 1 "GND" H 7075 3775 50  0001 C CNN
 F 2 "" H 7075 3925 50  0001 C CNN
@@
 Connection ~ 6725 3875
 $Comp
-L RF_Connectors:SMA_PCB J?
+L RF_Connectors:SMA_PCB J202
 U 1 1 5B3C280A
 P 8425 3400
-F 0 "J?" H 8400 3550 60  0000 C CNN
+F 0 "J202" H 8400 3550 60  0000 C CNN
 F 1 "SMA_PCB" H 8425 3600 60  0001 C CNN
 F 2 "Connectors_RF:PAD_T_200x110um" H 8425 3400 60  0001 C CNN
@@
 $EndComp
 $Comp
-L passives:CAP_0402 C?
+L passives:CAP_0402 C209
 U 1 1 5B3C280C
 P 8075 3950
-F 0 "C?" H 7975 4000 25  0000 C CNN
+F 0 "C209" H 7975 4000 25  0000 C CNN
 F 1 "22pF" H 8075 4050 25  0000 C CNN
 F 2 "SM0402" H 8075 4050 60  0001 C CNN
@@
 	8250 3950 8175 3950
 $Comp
-L power:GND #PWR?
+L power:GND #PWR0160
 U 1 1 5B3C280D
 P 8575 3550
-F 0 "#PWR?" H 8575 3300 50  0001 C CNN
+F 0 "#PWR0160" H 8575 3300 50  0001 C CNN
 F 1 "GND" H 8575 3400 50  0001 C CNN
 F 2 "" H 8575 3550 50  0001 C CNN
@@
 Connection ~ 7025 3875
 $Comp
-L passives:IND_0603 L?
+L passives:IND_0603 L203
 U 1 1 5B3C2830
 P 6875 3050
-F 0 "L?" H 6975 3100 25  0000 C CNN
+F 0 "L203" H 6975 3100 25  0000 C CNN
 F 1 "IND_0603" H 6825 3100 25  0000 C CNN
 F 2 "SM0603" H 6875 3050 60  0001 C CNN
@@
 	6875 3150 6875 3200
 $Comp
-L passives:IND_0603 L?
+L passives:IND_0603 L202
 U 1 1 5A02D2F6
 P 6775 3050
-F 0 "L?" H 6875 3100 25  0000 C CNN
+F 0 "L202" H 6875 3100 25  0000 C CNN
 F 1 "IND_0603" H 6725 3100 25  0000 C CNN
 F 2 "SM0603" H 6775 3050 60  0001 C CNN
@@
 $EndComp
 $Comp
-L passives:IND_0603 L?
+L passives:IND_0603 L201
 U 1 1 5B3C2832
 P 6675 3050
-F 0 "L?" H 6775 3100 25  0000 C CNN
+F 0 "L201" H 6775 3100 25  0000 C CNN
 F 1 "IND_0603" H 6625 3100 25  0000 C CNN
 F 2 "SM0603" H 6675 3050 60  0001 C CNN
@@
 	6675 3150 6675 3250
 $Comp
-L passives:CAP_0402 C?
+L passives:CAP_0402 C204
 U 1 1 5B3C2811
 P 7125 2900
-F 0 "C?" H 7125 2800 25  0000 C CNN
+F 0 "C204" H 7125 2800 25  0000 C CNN
 F 1 "47pF" H 7125 2975 25  0000 C CNN
 F 2 "SM0402" H 7125 3000 60  0001 C CNN
@@
 $EndComp
 $Comp
-L passives:CAP_0402 C?
+L passives:CAP_0402 C205
 U 1 1 5B3C2812
 P 7125 3200
-F 0 "C?" H 7125 3100 25  0000 C CNN
+F 0 "C205" H 7125 3100 25  0000 C CNN
 F 1 "22pF" H 7125 3275 25  0000 C CNN
 F 2 "SM0402" H 7125 3300 60  0001 C CNN
@@
 Connection ~ 6875 3200
 $Comp
-L power:GND #PWR?
+L power:GND #PWR0161
 U 1 1 5B3C2813
 P 7275 3250
-F 0 "#PWR?" H 7275 3000 50  0001 C CNN
+F 0 "#PWR0161" H 7275 3000 50  0001 C CNN
 F 1 "GND" H 7275 3100 50  0001 C CNN
 F 2 "" H 7275 3250 50  0001 C CNN
@@
 Connection ~ 7275 2900
 $Comp
-L passives:CAP_0402 C?
+L passives:CAP_0402 C208
 U 1 1 5A1BAA32
 P 7900 4125
-F 0 "C?" H 7900 4025 25  0000 C CNN
+F 0 "C208" H 7900 4025 25  0000 C CNN
 F 1 "0.15pF" H 7900 4200 25  0000 C CNN
 F 2 "SM0402" H 7900 4225 60  0001 C CNN
@@
 $EndComp
 $Comp
-L power:GND #PWR?
+L power:GND #PWR0162
 U 1 1 5B3C2816
 P 7900 4300
-F 0 "#PWR?" H 7900 4050 50  0001 C CNN
+F 0 "#PWR0162" H 7900 4050 50  0001 C CNN
 F 1 "GND" H 7900 4150 50  0001 C CNN
 F 2 "" H 7900 4300 50  0001 C CNN
@@
 Connection ~ 7900 3950
 $Comp
-L passives:CAP_0402 C?
+L passives:CAP_0402 C206
 U 1 1 5A02D301
 P 7675 3150
-F 0 "C?" H 7675 3050 25  0000 C CNN
+F 0 "C206" H 7675 3050 25  0000 C CNN
 F 1 "0.15pF" H 7675 3225 25  0000 C CNN
 F 2 "SM0402" H 7675 3250 60  0001 C CNN
@@
 Connection ~ 7675 3400
 $Comp
-L power:GND #PWR?
+L power:GND #PWR0163
 U 1 1 5B3C2818
 P 7675 2950
-F 0 "#PWR?" H 7675 2700 50  0001 C CNN
+F 0 "#PWR0163" H 7675 2700 50  0001 C CNN
 F 1 "GND" H 7675 2800 50  0001 C CNN
 F 2 "" H 7675 2950 50  0001 C CNN
@@
 Wire Wire Line
 	7000 2675 7000 2900
-$Comp
-L power:+3.3VA #PWR?
-U 1 1 5C6148D0
-P 7000 2450
-F 0 "#PWR?" H 7000 2300 50  0001 C CNN
-F 1 "+3.3VA" H 7050 2650 50  0000 C CNN
-F 2 "" H 7000 2450 50  0001 C CNN
-F 3 "" H 7000 2450 50  0001 C CNN
-	1    7000 2450
-	1    0    0    -1
-$EndComp
 Text Label 8050 3400 0    25   ~ 0
 R1_0
@@
 	7775 3400 7675 3400
 $Comp
-L passives:CAP_0402 C?
+L passives:CAP_0402 C207
 U 1 1 5B3C282E
 P 7875 3400
-F 0 "C?" H 7775 3450 25  0000 C CNN
+F 0 "C207" H 7775 3450 25  0000 C CNN
 F 1 "22pF" H 7875 3500 25  0000 C CNN
 F 2 "SM0402" H 7875 3500 60  0001 C CNN
@@
 	7475 3350 7475 2650
 $Comp
-L ltc5548:LTC5549 U?
+L ltc5548:LTC5549 U201
 U 1 1 5F7A86DC
 P 6825 3400
-F 0 "U?" H 6375 3150 60  0000 L CNN
+F 0 "U201" H 6375 3150 60  0000 L CNN
 F 1 "LTC5549" H 6725 2825 60  0000 L CNN
 F 2 "QFN:QFN12_2x3mm_UDB_LT" H 6825 3400 60  0001 C CNN
@@
 Connection ~ 6625 3875
 $Comp
-L passives:CAP_0402 C?
+L passives:CAP_0402 C202
 U 1 1 5F7AB513
 P 6175 3400
-F 0 "C?" H 6075 3450 25  0000 C CNN
+F 0 "C202" H 6075 3450 25  0000 C CNN
 F 1 "30pF" H 6250 3500 25  0000 C CNN
 F 2 "SM0402" H 6175 3500 60  0001 C CNN
@@
 	6275 3400 6425 3400
 $Comp
-L minic_bfcw:BFCW F?
+L minic_bfcw:BFCW F201
 U 1 1 5F7AC9E3
 P 5600 3400
-F 0 "F?" H 5600 3650 39  0000 C CNN
+F 0 "F201" H 5600 3650 39  0000 C CNN
 F 1 "BFCW-542+" H 5600 3550 39  0000 C CNN
 F 2 "" H 5600 3400 50  0001 C CNN
@@
 	5900 3400 6075 3400
 $Comp
-L power:GND #PWR?
+L power:GND #PWR0164
 U 1 1 5F7ADF38
 P 5500 3700
-F 0 "#PWR?" H 5500 3450 50  0001 C CNN
+F 0 "#PWR0164" H 5500 3450 50  0001 C CNN
 F 1 "GND" H 5500 3550 50  0001 C CNN
 F 2 "" H 5500 3700 50  0001 C CNN
@@
 	5500 3650 5500 3700
 $Comp
-L RF_Connectors:SMA_PCB J?
+L RF_Connectors:SMA_PCB J201
 U 1 1 5F7B1843
 P 4475 3400
-F 0 "J?" H 4450 3550 60  0000 C CNN
+F 0 "J201" H 4450 3550 60  0000 C CNN
 F 1 "SMA_PCB" H 4475 3600 60  0001 C CNN
 F 2 "Connectors_RF:PAD_T_200x110um" H 4475 3400 60  0001 C CNN
@@
 	5300 3400 5150 3400
 $Comp
-L power:GND #PWR?
+L power:GND #PWR0165
 U 1 1 5F7B3211
 P 4400 3600
-F 0 "#PWR?" H 4400 3350 50  0001 C CNN
+F 0 "#PWR0165" H 4400 3350 50  0001 C CNN
 F 1 "GND" H 4400 3450 50  0001 C CNN
 F 2 "" H 4400 3600 50  0001 C CNN
@@
 	4400 3475 4400 3600
 $Comp
-L passives:CAP_0603 C?
+L passives:CAP_0603 C203
 U 1 1 5F7B6AFE
 P 7125 2675
-F 0 "C?" H 7125 2600 25  0000 C CNN
+F 0 "C203" H 7125 2600 25  0000 C CNN
 F 1 "1uF" H 7125 2750 25  0000 C CNN
 F 2 "SM0603" H 7125 2775 60  0001 C CNN
@@
 $EndComp
 $Comp
-L passives:CAP_0402 C?
+L passives:CAP_0402 C201
 U 1 1 5F7C11DF
 P 5050 3400
-F 0 "C?" H 4950 3450 25  0000 C CNN
+F 0 "C201" H 4950 3450 25  0000 C CNN
 F 1 "30pF" H 5125 3500 25  0000 C CNN
 F 2 "SM0402" H 5050 3500 60  0001 C CNN
@@
 Wire Wire Line
 	4625 3400 4950 3400
+$Comp
+L power_symbols:+3.3VM1 #PWR0166
+U 1 1 5F9FEA59
+P 7000 2450
+F 0 "#PWR0166" H 7000 2410 30  0001 C CNN
+F 1 "+3.3VM1" H 7050 2600 30  0000 C CNN
+F 2 "" H 7000 2450 60  0000 C CNN
+F 3 "" H 7000 2450 60  0000 C CNN
+	1    7000 2450
+	1    0    0    -1
+$EndComp
 $EndSCHEMATC

Commit message: sent in production
Parts:
- F201: footprint (none) -> MiniCircuits:JC0603C
Changed lines of the file:
@@
 U 1 1 5F7A86DC
 P 6825 3400
-F 0 "U201" H 6375 3150 60  0000 L CNN
+F 0 "U201" V 7200 3100 60  0000 L CNN
 F 1 "LTC5549" H 6725 2825 60  0000 L CNN
 F 2 "QFN:QFN12_2x3mm_UDB_LT" H 6825 3400 60  0001 C CNN
@@
 F 0 "F201" H 5600 3650 39  0000 C CNN
 F 1 "BFCW-542+" H 5600 3550 39  0000 C CNN
-F 2 "" H 5600 3400 50  0001 C CNN
+F 2 "MiniCircuits:JC0603C" H 5600 3400 50  0001 C CNN
 F 3 "" H 5600 3400 50  0001 C CNN
 	1    5600 3400
